Commit message: Colission added and new manipulator file

File: ros2_ur3_project/workspace/custom_code/custom_ur_description/urdf/ALT_CUSTOM_station_macro.xacro (robot description, xacro)
@@ -24,10 +24,10 @@
 		<visual>
 			<origin xyz="0 0 0" rpy="0 0 0"/>
-			<geometry><box size="0.6 0.9 1"/></geometry>
+			<geometry><box size="${size} ${size} ${height}"/></geometry>
 			<material name="station_mat"><color rgba="${rgba_grey}"/></material>
 		</visual>
 		<collision>
 			<origin xyz="0 0 0" rpy="0 0 0"/>
-			<geometry><box size="0.6 0.9 1"/></geometry>
+			<geometry><box size="${size} ${size} ${height}"/></geometry>
 		</collision>
 	</link>
@@ -36,5 +36,5 @@
 			<child  link="station_cube"/>
 			<!-- hebt den Würfel um height/2, sodass seine Unterseite bei station.z=0 liegt -->
-			<origin xyz="${0.5*0.6} ${0.5*0.9} ${-0.5*1}" rpy="0 0 0"/>
+			<origin xyz="${0.5*size} ${0.5*size} ${-0.5*height}" rpy="0 0 0"/>
 	  	</joint>
   <!-- Definiert station_top, dort wird der Roboter gemountet -->
@@ -43,28 +43,12 @@
 			<parent link="station"/>
 			<child  link="station_top"/>
-			<origin xyz="0.225 0.325 0.02" rpy="0 0 1.5708"/>
+			<origin xyz="0.25 0.25 0.06" rpy="0 0 1.5708"/>
 		</joint>
-	<!-- Zylinder: Mittelpunkt (0.05, 0.08, 0.02), Höhe 0.9, Durchmesser 0.06 -->
-	<link name="custom_cylinder">
-		<visual>
-			<origin xyz="0 0 0" rpy="0 0 0"/>
-			<geometry><cylinder length="0.9" radius="0.03"/></geometry>
-			<material name="cylinder_mat"><color rgba="0.7 0.7 0.2 1.0"/></material>
-		</visual>
-		<collision>
-			<origin xyz="0 0 0" rpy="0 0 0"/>
-			<geometry><cylinder length="0.9" radius="0.03"/></geometry>
-		</collision>
-	</link>
-		<joint name="station_cube_to_custom_cylinder" type="fixed">
-			<parent link="station_cube"/>
-			<child link="custom_cylinder"/>
-			<!-- Oberseite von station_cube: z=1, Zylinder steht mit Unterseite darauf -->
-			<origin xyz="-0.25 0.40 1.0" rpy="0 0 0"/>
-		</joint>
-  <!-- Erstellt 2 Platten auf der Station aus der Macro -->
+  <!-- Erstellt 4 Platten auf der Station aus der Macro -->
 	<xacro:include filename="$(find custom_ur_description)/urdf/CUSTOM_elementary_unit_macro.xacro"/>
-		<xacro:elementary_unit prefix="u1" size_x="0.25" size_y="0.25" height="0.02" pos_on_station="0.1 0.2" rgba="${rgba_black}"/>
-		<xacro:elementary_unit prefix="u4" size_x="0.25" size_y="0.45" height="0.02" pos_on_station="0.35 0.45" rgba="${rgba_blue}"/>
+		<xacro:elementary_unit prefix="u1" pos_on_station="0.0 0.0" rgba="${rgba_black}"/>
+		<xacro:elementary_unit prefix="u2" pos_on_station="0.5 0.0" rgba="${rgba_blue}"/>
+		<xacro:elementary_unit prefix="u3" pos_on_station="0.0 0.5" rgba="${rgba_blue}"/>
+		<xacro:elementary_unit prefix="u4" pos_on_station="0.5 0.5" rgba="${rgba_blue}"/>
 	</xacro:macro>
 </robot>

File: ros2_ur3_project/workspace/custom_code/custom_ur_description/urdf/CUSTOM_elementary_unit_macro.xacro (robot description, xacro)
@@ -3,10 +3,11 @@
   <!-- Macro: erzeugt eine quadratische Elementareinheit, für die 4 gleichen Platten -->
   <xacro:macro name="elementary_unit" params="
-      prefix
-      parent:=station
-      size:=0.5
-      height:=0.06
-      pos_on_station:= '0 0'
-      rgba:='0.0 0.0 0.0 1.0'">
+    prefix
+    parent:=station
+    size_x:=0.5
+    size_y:=0.5
+    height:=0.06
+    pos_on_station:='0 0'
+    rgba:='0.0 0.0 0.0 1.0'">
       <link name="${prefix}_KOS"/>
         <joint name="${prefix}_to_parent" type="fixed">
@@ -18,16 +19,16 @@
         <visual>
           <origin xyz="0 0 0" rpy="0 0 0"/>
-            <geometry><box size="${size} ${size} ${height}"/></geometry>
+            <geometry><box size="${size_x} ${size_y} ${height}"/></geometry>
             <material name="${prefix}_e_mat"><color rgba="${rgba}"/></material>
         </visual>
         <collision>
           <origin xyz="0 0 0" rpy="0 0 0"/>
-          <geometry><box size="${size} ${size} ${height}"/></geometry>
+          <geometry><box size="${size_x} ${size_y} ${height}"/></geometry>
         </collision>
       </link>
       <joint name="${prefix}_kos_cube" type="fixed">
-	      <parent link="${prefix}_KOS"/>
-	      <child  link="${prefix}_cube"/>
-	      <origin xyz="${0.5*size} ${0.5*size} ${0.5*height}" rpy="0 0 0"/>
+        <parent link="${prefix}_KOS"/>
+        <child  link="${prefix}_cube"/>
+        <origin xyz="${0.5*size_x} ${0.5*size_y} ${0.5*height}" rpy="0 0 0"/>
       </joint>
   </xacro:macro>
