Commit message: Added gripper and acutal table model Moved tcp to gripper tip Removed collision disable between base and table to avoid unwanted collisions

File: ros2_ur3_project/workspace/custom_code/custom_ur_description/urdf/CUSTOM_elementary_unit_macro.xacro (robot description, xacro)
@@ -8,5 +8,5 @@
     size_y:=0.5
     height:=0.06
-    pos_on_station:='0 0'
+    pos_on_station:='0 0 0'
     rgba:='0.0 0.0 0.0 1.0'">
       <link name="${prefix}_KOS"/>
@@ -14,5 +14,5 @@
           <parent link="${parent}"/>
           <child  link="${prefix}_KOS"/>
-          <origin xyz="${pos_on_station} 0" rpy="0 0 0"/>
+          <origin xyz="${pos_on_station}" rpy="0 0 0"/>
         </joint>
       <link name="${prefix}_cube">

File: ros2_ur3_project/workspace/custom_code/custom_ur_description/urdf/CUSTOM_station_macro.xacro (robot description, xacro)
@@ -6,5 +6,5 @@
     parent:=world
     size:=1.0
-    height:=1.0
+    height:=0.92
 	robot_mount_xy:='1.0 1.0'
 	robot_mount_z:=1.0
@@ -12,5 +12,8 @@
 	rgba_grey:='0.4 0.4 0.4 0.5'
 	rgba_blue:='0.0 0.0 1.0 0.5'
-	rgba_black:='0.0 0.0 0.0 0.5'">
+	rgba_black:='0.0 0.0 0.0 0.8'
+	rgba_pink:='0.82 0.82 1.0 0.8'
+	rgba_light_grey:='0.8 0.8 0.8 1.0'
+	rgba_dark_grey:='0.6 0.6 0.6 1.0'">
   <!-- Bindet Station an world -->
 	<link name="station"/>
@@ -20,14 +23,14 @@
 	    <origin xyz="0 0 ${height}" rpy="0 0 0"/>
 	</joint>
-  <!-- Erstellt den Tisch, unterer Quader -->
+  <!-- Erstellt Tisch, unterer Quader -->
 	<link name="station_cube">
 		<visual>
 			<origin xyz="0 0 0" rpy="0 0 0"/>
-			<geometry><box size="0.6 0.9 1"/></geometry>
+			<geometry><box size="0.62 0.81 ${height}"/></geometry>
 			<material name="station_mat"><color rgba="${rgba_grey}"/></material>
 		</visual>
 		<collision>
 			<origin xyz="0 0 0" rpy="0 0 0"/>
-			<geometry><box size="0.6 0.9 1"/></geometry>
+			<geometry><box size="0.62 0.81 ${height}"/></geometry>
 		</collision>
 	</link>
@@ -36,35 +39,41 @@
 			<child  link="station_cube"/>
 			<!-- hebt den Würfel um height/2, sodass seine Unterseite bei station.z=0 liegt -->
-			<origin xyz="${0.5*0.6} ${0.5*0.9} ${-0.5*1}" rpy="0 0 0"/>
+			<origin xyz="${0.5*0.62} ${0.5*0.81} ${-0.5*height}" rpy="0 0 0"/>
 	  	</joint>
   <!-- Definiert station_top, dort wird der Roboter gemountet -->
 	<link name="station_top"/>
-		<joint name="station_to_top" type="fixed">
-			<parent link="station"/>
+		<joint name="u1_cube_to_top" type="fixed">
+			<parent link="u1_cube"/>
 			<child  link="station_top"/>
-			<origin xyz="0.225 0.325 0.02" rpy="0 0 1.5708"/>
+			<origin xyz="0 0 0.013" rpy="0 0 1.5708"/>
 		</joint>
-	<!-- Zylinder: Mittelpunkt (0.05, 0.08, 0.02), Höhe 0.9, Durchmesser 0.06 -->
+	<!-- Zylinder: Mittelpunkt (0.05, 0.08, 0.02), Höhe 0.643, Durchmesser 0.06 -->
 	<link name="custom_cylinder">
 		<visual>
 			<origin xyz="0 0 0" rpy="0 0 0"/>
-			<geometry><cylinder length="0.9" radius="0.03"/></geometry>
-			<material name="cylinder_mat"><color rgba="0.7 0.7 0.2 1.0"/></material>
+			<geometry><cylinder length="0.643" radius="0.0225"/></geometry>
+			<material name="cylinder_mat"><color rgba="${rgba_black}"/></material>
 		</visual>
 		<collision>
 			<origin xyz="0 0 0" rpy="0 0 0"/>
-			<geometry><cylinder length="0.9" radius="0.03"/></geometry>
+			<geometry><cylinder length="0.643" radius="0.0225"/></geometry>
 		</collision>
 	</link>
-		<joint name="station_cube_to_custom_cylinder" type="fixed">
-			<parent link="station_cube"/>
+		<joint name="top_plate_cube_to_custom_cylinder" type="fixed">
+			<parent link="top_plate_cube"/>
 			<child link="custom_cylinder"/>
-			<!-- Oberseite von station_cube: z=1, Zylinder steht mit Unterseite darauf -->
-			<origin xyz="-0.25 0.40 1.0" rpy="0 0 0"/>
+			<!-- Oberseite von top_plate_cube: z=1.02, Zylinder steht mit Unterseite darauf -->
+			<origin xyz="-0.205 0.36 0.325" rpy="0 0 0"/>
 		</joint>
   <!-- Erstellt 2 Platten auf der Station aus der Macro -->
 	<xacro:include filename="$(find custom_ur_description)/urdf/CUSTOM_elementary_unit_macro.xacro"/>
-		<xacro:elementary_unit prefix="u1" size_x="0.25" size_y="0.25" height="0.02" pos_on_station="0.1 0.2" rgba="${rgba_black}"/>
-		<xacro:elementary_unit prefix="u4" size_x="0.25" size_y="0.45" height="0.02" pos_on_station="0.35 0.45" rgba="${rgba_blue}"/>
+		<xacro:elementary_unit prefix="u1" size_x="0.25" size_y="0.25" height="0.026" pos_on_station="0.12 0.155 0.02" rgba="${rgba_dark_grey}"/>
+		<xacro:elementary_unit prefix="u4" size_x="0.25" size_y="0.405" height="0.026" pos_on_station="0.37 0.405 0.02" rgba="${rgba_light_grey}"/>
+		<!-- Platte mit den Maßen der station_cube (0.6 x 0.9), 2cm dick, auf station_cube oben drauf -->
+		<xacro:elementary_unit prefix="top_plate" size_x="0.62" size_y="0.81" height="0.02" pos_on_station="0 0 0" rgba="${rgba_pink}"/>
+		<xacro:elementary_unit prefix="wbk1" size_x="0.2" size_y="0.2" height="0.06" pos_on_station="0.395 0.18 0.02" rgba="${rgba_black}"/>
+		<xacro:elementary_unit prefix="wbk12" size_x="0.06" size_y="0.06" height="0.12" pos_on_station="0.495 0.28 0.08" rgba="${rgba_black}"/>
+		<xacro:elementary_unit prefix="wbk2" size_x="0.2" size_y="0.2" height="0.06" pos_on_station="0.145 0.42 0.02" rgba="${rgba_black}"/>
+		<xacro:elementary_unit prefix="wbk22" size_x="0.06" size_y="0.06" height="0.12" pos_on_station="0.245 0.52 0.08" rgba="${rgba_black}"/>
 	</xacro:macro>
 </robot>

File: ros2_ur3_project/workspace/custom_code/custom_ur_description/urdf/CUSTOM_ur3e.urdf.xacro (robot description, xacro)
@@ -4,5 +4,6 @@
    <xacro:arg name="name" default="ur3"/>
    <!-- import main macro -->
-   <xacro:include filename="$(find custom_ur_description)/urdf/ur_macro.xacro"/>
+  <xacro:include filename="$(find custom_ur_description)/urdf/ur_macro.xacro"/>
+  <xacro:include filename="$(find custom_ur_description)/urdf/CUSTOM_gripper_macro.xacro"/>
    <!-- ur_type: ur3 -->
    <xacro:arg name="ur_type" default="ur3"/>
@@ -105,3 +106,6 @@
      <origin xyz="0 0 0" rpy="0 0 3.141" />
    </xacro:ur_robot>
+  <!-- Adapterflansch und EGP-C 40 Gripper (Makros)
+  <xacro:ur3e_adapterflange parent_link="tool0"/>-->
+  <xacro:egpc40_gripper parent_link="tool0"/>
 </robot>

File: ros2_ur3_project/workspace/custom_code/custom_ur_moveit_config/srdf/ur.srdf.xacro (robot description, xacro)
@@ -3,6 +3,7 @@
   <!-- MoveIt SRDF for UR3 -->
   <group name="ur_manipulator">
-    <chain base_link="base_link" tip_link="tool0" />
+    <chain base_link="base_link" tip_link="tcp" />
   </group>
+  <!-- TCP als Endeffektor für MoveIt -->
   <group_state name="home" group="ur_manipulator">
     <joint name="elbow_joint" value="0" />
@@ -13,6 +14,7 @@
     <joint name="wrist_3_joint" value="0" />
   </group_state>
+  <!-- Virtual Joint to attach the robot to the world -->
   <virtual_joint name="world_joint" type="fixed" parent_frame="world" child_link="base_link"/>
-  <disable_collisions link1="base_link" link2="base_link_inertia" reason="Adjacent" />
+  <!-- Disable collisions for the robot -->
   <disable_collisions link1="base_link_inertia" link2="shoulder_link" reason="Adjacent" />
   <disable_collisions link1="tool0" link2="wrist_1_link" reason="Never" />
@@ -25,26 +27,18 @@
   <disable_collisions link1="wrist_1_link" link2="wrist_3_link" reason="Never" />
   <disable_collisions link1="wrist_2_link" link2="wrist_3_link" reason="Adjacent" />
-  <disable_collisions link1="base_link" link2="station" reason="Never" />
-  <disable_collisions link1="base_link" link2="station_cube" reason="Never" />
-  <disable_collisions link1="base_link" link2="station_top" reason="Never" />
-  <disable_collisions link1="base_link" link2="robot_mount_cylinder" reason="Never" />
-  <disable_collisions link1="tool0" link2="station" reason="Never" />
-  <disable_collisions link1="tool0" link2="station_cube" reason="Never" />
-  <disable_collisions link1="tool0" link2="station_top" reason="Never" />
-  <disable_collisions link1="tool0" link2="robot_mount_cylinder" reason="Never" />
-  <!-- Kollisionen base_link_inertia mit station_cube und uX_cube deaktiviert -->
-  <disable_collisions link1="base_link_inertia" link2="station_cube" reason="Never" />
+  <!-- Disable collisions with added links -->
   <disable_collisions link1="base_link_inertia" link2="u1_cube" reason="Never" />
-  <disable_collisions link1="base_link_inertia" link2="u2_cube" reason="Never" />
-  <disable_collisions link1="base_link_inertia" link2="u3_cube" reason="Never" />
-  <disable_collisions link1="base_link_inertia" link2="u4_cube" reason="Never" />
-  <!-- Kollisionen zwischen Base und Tisch bleiben aktiv (aus ur_macro.srdf.xacro übernommen) -->
+  <disable_collisions link1="egpc40_gripper" link2="wrist_3_link" reason="Adjacent" />
+  <!-- Disable collisions between base and table  -->
   <disable_collisions link1="station_cube" link2="u1_cube" reason="Table" />
-  <disable_collisions link1="station_cube" link2="u2_cube" reason="Table" />
-  <disable_collisions link1="station_cube" link2="u3_cube" reason="Table" />
   <disable_collisions link1="station_cube" link2="u4_cube" reason="Table" />
-  <disable_collisions link1="u1_cube" link2="u2_cube" reason="Table" />
-  <disable_collisions link1="u1_cube" link2="u3_cube" reason="Table" />
-  <disable_collisions link1="u2_cube" link2="u4_cube" reason="Table" />
-  <disable_collisions link1="u3_cube" link2="u4_cube" reason="Table" />
+  <disable_collisions link1="station_cube" link2="top_plate_cube" reason="Table" />
+  <disable_collisions link1="top_plate_cube" link2="u1_cube" reason="Table" />
+  <disable_collisions link1="top_plate_cube" link2="u4_cube" reason="Table" />
+  <disable_collisions link1="top_plate_cube" link2="custom_cylinder" reason="Table" />
+  <disable_collisions link1="top_plate_cube" link2="wbk1_cube" reason="Table" />
+  <disable_collisions link1="top_plate_cube" link2="wbk2_cube" reason="Table" />
+  <disable_collisions link1="wbk1_cube" link2="wbk12_cube" reason="Table" />
+  <disable_collisions link1="wbk2_cube" link2="wbk22_cube" reason="Table" />
+  <disable_collisions link1="u1_cube" link2="u4_cube" reason="Table" />
 </robot>
