Commit message: Start_scipts updated and Dockerfile modified to build RTDE from source

File: ros2_ur3_project/workspace/custom_code/custom_ur_description/urdf/CUSTOM_gripper_macro.xacro (robot description, xacro)
@@ -21,7 +21,7 @@
     </link>
     <joint name="${parent_link}_to_egpc40_gripper" type="fixed">
-      <parent link="${parent_link}"/>
-      <child link="egpc40_gripper"/>
-      <origin xyz="0 0 0.118" rpy="0 0 0"/>
+  <parent link="${parent_link}"/>
+  <child link="egpc40_gripper"/>
+  <origin xyz="0 0 0.118" rpy="0 0 -0.7854"/>
     </joint>
   </xacro:macro>

Commit message: roboter moves to predefined grip position and grips there, currently above the toolhead

File: ros2_ur3_project/workspace/custom_code/custom_ur_description/urdf/CUSTOM_gripper_macro.xacro (robot description, xacro)
@@ -5,7 +5,7 @@
     <link name="egpc40_gripper">
       <visual>
-        <origin xyz="0 0 0" rpy="0 0 0"/>
+        <origin xyz="0 0 0" rpy="0 0 3.1416"/>
         <geometry>
-          <mesh filename="package://custom_ur_description/meshes/CUSTOM_meshes/SCHUNK-Gripper-Fingers.stl"/>
+          <mesh filename="package://custom_ur_description/meshes/CUSTOM_meshes/SCHUNK-Gripper-Fingers.stl" scale="0.001 0.001 0.001"/>
         </geometry>
         <material name="blue">
@@ -14,7 +14,7 @@
       </visual>
       <collision>
-        <origin xyz="0 0 0" rpy="0 0 0"/>
+        <origin xyz="0 0 0" rpy="0 0 3.1416"/>
         <geometry>
-          <mesh filename="package://custom_ur_description/meshes/CUSTOM_meshes/SCHUNK-Gripper-Fingers.stl"/>
+          <mesh filename="package://custom_ur_description/meshes/CUSTOM_meshes/SCHUNK-Gripper-Fingers.stl" scale="0.00105 0.00105 0.00105"/>
         </geometry>
       </collision>
@@ -31,5 +31,5 @@
         <parent link="egpc40_gripper"/>
         <child link="tcp"/>
-        <origin xyz="0 0 0.05" rpy="0 0 0"/>
+        <origin xyz="0 0 0.0375" rpy="0 0 0"/>
     </joint>
 </robot>
