Commit message: connected the two docker, works fine with real movement; detects the plier and moves above it

File: ros2_ur3_project/workspace/custom_code/custom_ur_description/urdf/CUSTOM_station_macro.xacro (robot description, xacro)
@@ -10,4 +10,5 @@
 	robot_mount_z:=1.0
 	robot_mount_yaw:=0.0
+	aruco_on_station:='0.0 0.81 0.02'
 	rgba_grey:='0.4 0.4 0.4 0.5'
 	rgba_blue:='0.0 0.0 1.0 0.5'
@@ -78,4 +79,12 @@
 		<!-- Wand -->
 		<xacro:elementary_unit prefix="wall" size_x="0.02" size_y="0.35" height="0.45" pos_on_station="0 0.46 0.02" rgba="${rgba_black}"/>
+		<!-- Fester Referenz-Frame fuer den ArUco-Ursprung auf der Tischoberseite. -->
+		<!-- Wichtig: Nicht 'aruco_0' nennen, um keinen TF-Konflikt mit dem D405-Tracker zu erzeugen. -->
+		<link name="aruco_table_ref_0"/>
+		<joint name="station_to_aruco_table_ref_0" type="fixed">
+			<parent link="station"/>
+			<child  link="aruco_table_ref_0"/>
+			<origin xyz="${aruco_on_station}" rpy="0 0 0"/>
+		</joint>
 	</xacro:macro>
 </robot>

Commit message: works good, new environment

File: ros2_ur3_project/workspace/custom_code/custom_ur_description/urdf/CUSTOM_station_macro.xacro (robot description, xacro)
@@ -75,8 +75,6 @@
 		<xacro:elementary_unit prefix="wbk1" size_x="0.2" size_y="0.2" height="0.06" pos_on_station="0.395 0.18 0.02" rgba="${rgba_black}"/>
 		<xacro:elementary_unit prefix="wbk12" size_x="0.06" size_y="0.06" height="0.12" pos_on_station="0.495 0.28 0.08" rgba="${rgba_black}"/>
-		<xacro:elementary_unit prefix="wbk2" size_x="0.2" size_y="0.2" height="0.06" pos_on_station="0.145 0.42 0.02" rgba="${rgba_black}"/>
-		<xacro:elementary_unit prefix="wbk22" size_x="0.06" size_y="0.06" height="0.12" pos_on_station="0.245 0.52 0.08" rgba="${rgba_black}"/>
-		<!-- Wand -->
-		<xacro:elementary_unit prefix="wall" size_x="0.02" size_y="0.35" height="0.45" pos_on_station="0 0.46 0.02" rgba="${rgba_black}"/>
+		<!-- <xacro:elementary_unit prefix="wbk2" size_x="0.2" size_y="0.2" height="0.06" pos_on_station="0.145 0.42 0.02" rgba="${rgba_black}"/> -->
+		<!-- <xacro:elementary_unit prefix="wbk22" size_x="0.06" size_y="0.06" height="0.12" pos_on_station="0.245 0.52 0.08" rgba="${rgba_black}"/> -->
 		<!-- Fester Referenz-Frame fuer den ArUco-Ursprung auf der Tischoberseite. -->
 		<!-- Wichtig: Nicht 'aruco_0' nennen, um keinen TF-Konflikt mit dem D405-Tracker zu erzeugen. -->
@@ -87,4 +85,25 @@
 			<origin xyz="${aruco_on_station}" rpy="0 0 0"/>
 		</joint>
+		<!-- Zangenablage -->
+		<link name="zangenablage">
+			<visual>
+				<origin xyz="0 0 0" rpy="0 0 0"/>
+				<geometry>
+					<mesh filename="package://custom_ur_description/meshes/CUSTOM_meshes/Ablageflaeche-und-Schraege-V1.stl" scale="1 1 1"/>
+				</geometry>
+				<material name="zangenablage_mat"><color rgba="0.6 0.6 0.6 1.0"/></material>
+			</visual>
+			<collision>
+				<origin xyz="0 0 0" rpy="0 0 0"/>
+				<geometry>
+					<mesh filename="package://custom_ur_description/meshes/CUSTOM_meshes/Ablageflaeche-und-Schraege-V1.stl" scale="1 1 1"/>
+				</geometry>
+			</collision>
+		</link>
+		<joint name="station_to_zangenablage" type="fixed">
+			<parent link="station"/>
+			<child  link="zangenablage"/>
+			<origin xyz="0.37 0.4 0.02" rpy="0 0 1.5708"/>
+		</joint>
 	</xacro:macro>
 </robot>

File: ros2_ur3_project/workspace/custom_code/custom_ur_moveit_config/srdf/ur.srdf.xacro (robot description, xacro)
@@ -38,7 +38,6 @@
   <disable_collisions link1="top_plate_cube" link2="custom_cylinder" reason="Table" />
   <disable_collisions link1="top_plate_cube" link2="wbk1_cube" reason="Table" />
-  <disable_collisions link1="top_plate_cube" link2="wbk2_cube" reason="Table" />
   <disable_collisions link1="wbk1_cube" link2="wbk12_cube" reason="Table" />
-  <disable_collisions link1="wbk2_cube" link2="wbk22_cube" reason="Table" />
+  <disable_collisions link1="top_plate_cube" link2="zangenablage" reason="Table" />
   <disable_collisions link1="u1_cube" link2="u4_cube" reason="Table" />
 </robot>
